File: CM4-Interposer.brd (EAGLE design)
At the start: 55 x 40 mm, 2 parts

Commit message: misc
Parts:
- added U$3: (no value), Custom-Parts:DIODES-DELIGHT-LOGO-15X15-BTM
Changed lines of the file:
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@@
 <attribute name="VALUE" x="26.17" y="24.78" size="1.27" layer="27" align="center"/>
 </element>
+<element name="U$3" library="Custom-Parts" library_urn="urn:adsk.eagle:library:25097078" package="DIODES-DELIGHT-LOGO-15X15-BTM" package3d_urn="urn:adsk.eagle:package:26399217/1" value="" x="36" y="16" smashed="yes" rot="MR0"/>
 </elements>
 <signals>
